File: Blue_Wizard/Blue_Wizard.kicad_pcb (KiCad board)
At the start: 2 copper layers, 120.6 x 95.2 mm, 37 parts, among them J1 Conn_ARM_JTAG_SWD_10, J10 Left Keywell Header, J11 Conn_01x02_Male, J12 10137062-00021LF, J13 Conn_01x01, J2 Conn_01x05, J3 Right FN, J4 Right Keywell, J5 Right Thumb Cluster, J6 Right Keywell Header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

Commit message: Rev 0 in progress
Parts:
- added C5: 10uf, Capacitor_SMD:C_0805_2012Metric, F.Cu at (165.1, 64.1)
- added C6: 0.1uf, Capacitor_SMD:C_0805_2012Metric, F.Cu at (156.2, 68.3)
- added C7: 0.1uf, Capacitor_SMD:C_0805_2012Metric, F.Cu at (149.1, 55.6)
- added C8: 1nF, Capacitor_SMD:C_0805_2012Metric, F.Cu at (117.3, 55.4)
- added J14: Conn_01x02, Connector_PinHeader_2.54mm:PinHeader_1x02_P2.54mm_Vertical, F.Cu at (105.9, 72.5)
- added R10: 100 ohm, Resistor_SMD:R_0805_2012Metric, F.Cu at (159.4, 55.9)
- added R11: 806k ohm, Resistor_SMD:R_0805_2012Metric, F.Cu at (115.3, 60.2)
- added R12: 2M, Resistor_SMD:R_0805_2012Metric, F.Cu at (117.3, 65.3)
- added U4: CP2104, Package_DFN_QFN:QFN-24-1EP_4x4mm_P0.5mm_EP2.6x2.6mm, F.Cu at (159.4, 62.2)
- added Y1: SIT1533AI-H4-DCC-32.768E, SamacSys_Parts:SIT1533AIH4DCC32768E, F.Cu at (128.0, 53.6)
- J11: value Conn_01x02_Male -> Conn_01x02
- R1, R2, R4: value 100 ohm -> 1k ohm
- R3: value 100 ohm -> 470 ohm
- U2: value MIC5504-3.3YM5 -> MIC5365-3.3YD5
- moved C1 15.7 mm to (109.7, 69.0)
- moved C2 13.7 mm to (115.1, 72.2)
- moved C3 11.7 mm to (185.5, 82.8)
- moved D5 2.79 mm to (125.2, 74.0)
- moved R5 2.79 mm to (125.2, 79.0)
- moved U2 2.68 mm to (110.4, 73.1)
Connections:
- net P6 renamed Net-(U1-PadP6)
- D1 pad 1: P8 -> Net-(D1-Pad1)
- D1 pad 2: Net-(D1-Pad2) -> LED2
- D2 pad 1: P7 -> Net-(D2-Pad1)
- D2 pad 2: Net-(D2-Pad2) -> LED1
- J12 pad A6: Net-(J12-PadA6) -> D+
- J12 pad A7: Net-(J12-PadA7) -> D-
- J12 pad B6: Net-(J12-PadB6) -> D+
- J12 pad B7: Net-(J12-PadB7) -> D-
- R1 pad 1: VCC -> GND
- R1 pad 2: Net-(D1-Pad2) -> Net-(D1-Pad1)
- R2 pad 1: VCC -> GND
- R2 pad 2: Net-(D2-Pad2) -> Net-(D2-Pad1)
- U1 pad P11: B5 -> B3
- U1 pad P12: B3 -> BMonitor
- U1 pad P14: Net-(U1-PadP14) -> GND
- U1 pad P22: D7 -> TXD
- U1 pad P23: C0 -> D7
- U1 pad P24: D6 -> RXD
- U1 pad P25: Net-(U1-PadP25) -> C0
- U1 pad P26: B6 -> D6
- U1 pad P27: Net-(U1-PadP27) -> B6
- U1 pad P35: D5 -> LED1
- U1 pad P37: B2 -> LED2
- U1 pad P7: P7 -> B2
- U1 pad P8: P8 -> D5
- U1 pad P9: Net-(U1-PadP9) -> B5
Routing:
- net P7: track 156.5 -> 0.00 mm
- net P8: track 145.1 -> 0.00 mm
- net LED2: track 0.00 -> 101.0 mm, vias 0 -> 4
- net D+: track 0.00 -> 94.3 mm, vias 0 -> 3
- net D-: track 0.00 -> 92.6 mm, vias 0 -> 2
- net LED1: track 0.00 -> 79.1 mm, vias 0 -> 2
- net B2: track 211.5 -> 261.4 mm, vias 0 -> 2
- net BMonitor: track 0.00 -> 46.5 mm
- net TXD: track 0.00 -> 39.7 mm, vias 0 -> 2
- net RXD: track 0.00 -> 32.3 mm, vias 0 -> 2
- net +BATT: track 104.3 -> 132.3 mm
- net B0: track 193.3 -> 220.4 mm, vias 3 -> 2
- net GND: track 48.8 -> 61.4 mm, vias 25 -> 32
- net DTR: track 0.00 -> 12.1 mm
- net Net-(U1-PadP14): track 11.4 -> 0.00 mm, vias 1 -> 0
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Other:
- board size 120.6 x 95.2 mm -> 108 x 95.2 mm
- board text added: "3.3V Enable"
- board text added: "Battery"
- board text added: "Battery Charging"
- board text added: "Battery Monitor"
- board text added: "Power Regulation"
- board text added: "USB/UART"
- board text added: "https://github.com/wizarddata/Blue-Wizard-Mod"
- board text added: "p.025"
- board text removed: "Blue Wizard Mod nRF52832 Modules - BMD-300 Vertical 13 Position - 0039532135 Horizontal 13 Position - 0039532134 Battery Management - MCP73831T-2ACI/OT LDO Reguator - MIC5504-3.3YM5-TR SWD Programming Header - 20021121-00010C4LF Reset Switch - PTS526 SK08 SMTR2 LFS USB C Jack - 10137062-00021LF Green 3mm LED - LTL-4231N"
- board text removed: "P11"
- board text removed: "P25"
- board text removed: "P28"
- board text removed: "P30"
- board text removed: "P31"
- board text removed: "R1 - R4 100 ohm R5 100k ohm R6 10k ohm R7 R8 5.1k ohm R9 2k ohm C1 C2 1uF C3 C4 4.7uF D5 MBR120"

Commit message: pre-final
Parts:
- D1, D2: moved to B.Cu
- D3: renamed from D4; moved to B.Cu
- D4: renamed from D3; moved to B.Cu
- moved R3 10.3 mm to (155.4, 116.8)
- moved R4 10.3 mm to (165.7, 116.8)
- moved D3 10.2 mm to (154.3, 124.5)
- moved D4 10.2 mm to (164.5, 124.5)
- renumbered R4 to R3, R3 to R4
Connections:
- C6 pad 1: VCC -> Net-(C6-Pad1)
- D1 pad 2: LED2 -> LED1
- D2 pad 2: LED1 -> LED2
- D3 pad 1: GND -> Net-(D3-Pad1)
- D3 pad 2: Net-(D4-Pad2) -> LED3
- R3 pad 1: +5V -> GND
- R3 pad 2: Net-(D4-Pad2) -> Net-(D3-Pad1)
- U1 pad P35: LED1 -> LED2
- U1 pad P37: LED2 -> LED1
- U1 pad P6: Net-(U1-PadP6) -> LED3
- U4 pad 5: VCC -> Net-(C6-Pad1)
- U4 pad 6: VCC -> Net-(C6-Pad1)
Routing:
- net LED3: track 0.00 -> 187.5 mm
- net Net-(R4-Pad1): track 63.7 -> 39.0 mm
- net LED2: track 101.0 -> 79.1 mm, vias 4 -> 2
- net LED1: track 79.1 -> 101.0 mm, vias 2 -> 4
- net Net-(D3-Pad1): track 0.00 -> 8.29 mm
- net Net-(D4-Pad2): track 7.21 -> 0.00 mm
- net VCC: track 66.8 -> 60.0 mm
- net Net-(C6-Pad1): track 0.00 -> 5.53 mm
- net +5V: track 227.3 -> 232.8 mm
- net Net-(U1-PadP6): track 3.93 -> 0.00 mm, vias 1 -> 0
- net B0: track 220.4 -> 218.3 mm
- net GND: track 61.4 -> 61.5 mm, vias 32 -> 33
Other:
- board text removed: "p.025"
