File: Blue_Wizard/Blue_Wizard.kicad_pcb (KiCad board)
At the start: 2 copper layers, 108 x 95.2 mm, 47 parts, among them J1 Conn_ARM_JTAG_SWD_10, J10 Left Keywell Header, J11 Conn_01x02, J12 10137062-00021LF, J13 Conn_01x01, J14 Conn_01x02, J2 Conn_01x05, J3 Right FN, J4 Right Keywell, J5 Right Thumb Cluster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

Commit message: readme update
Parts:
- removed J14: Conn_01x02, Connector_PinHeader_2.54mm:PinHeader_1x02_P2.54mm_Vertical
- U2: value MIC5365-3.3YD5 -> MIC5504-3.3YM5
- moved U2 0.15 mm to (110.5, 73.1)
Connections:
- U2 pad 3: Net-(J14-Pad2) -> Net-(C1-Pad1)
Routing:
- net B6: track 189.9 -> 206.7 mm
- net D5: track 156.3 -> 171.8 mm
- net B5: track 224.7 -> 236.3 mm
- net Net-(J14-Pad2): track 3.76 -> 0.00 mm
- net GND: track 61.5 -> 65.1 mm, vias 33 -> 35
- net Net-(C1-Pad1): track 30.4 -> 27.1 mm
Other:
- board text removed: "3.3V Enable"

Commit message: Final Gerbers and BOM
Parts:
- added J14: Conn_01x02, Connector_PinHeader_2.54mm:PinHeader_1x02_P2.54mm_Vertical, F.Cu at (105.6, 70.3)
Connections:
- U2 pad 3: Net-(C1-Pad1) -> Net-(J14-Pad2)
Routing:
- net Net-(J14-Pad2): track 0.00 -> 4.30 mm
- net +BATT: track 132.3 -> 136.1 mm
- net Net-(C1-Pad1): track 27.1 -> 29.5 mm

Commit message: Rev 0a board complete
Parts:
- moved J14 0.06 mm to (105.6, 70.4)
Connections:
- J7 pad 7: Net-(J7-Pad7) -> C6
Routing:
- net C6: track 179.4 -> 180.6 mm
