File: Blue_Wizard/Blue_Wizard.sch (KiCad schematic (older format))
At the start: 37 parts, among them J1 Conn_ARM_JTAG_SWD_10, J10 Left Keywell Header, J11 Conn_01x02_Male, J12 10137062-00021LF, J13 Conn_01x01, J2 Conn_01x05, J3 Right FN, J4 Right Keywell, J5 Right Thumb Cluster, J6 Right Keywell Header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

Commit message: Rev 0 in progress
Parts:
- removed U2: MIC5504-3.3YM5, Package_TO_SOT_SMD:SOT-23-5, symbol Regulator_Linear:MIC5504-1.8YM5
- added C5: 10uf, Capacitor_SMD:C_0805_2012Metric, symbol Device:C_Small
- added C6, C7: 0.1uf, Capacitor_SMD:C_0805_2012Metric, symbol Device:C_Small
- added C8: 1nF, Capacitor_SMD:C_0805_2012Metric, symbol Device:C_Small
- added J14: Conn_01x02, Connector_PinHeader_2.54mm:PinHeader_1x02_P2.54mm_Vertical, symbol Connector:Conn_01x02_Male
- added R10: 100 ohm, Resistor_SMD:R_0805_2012Metric, symbol Device:R_Small
- added R11: 806k ohm, Resistor_SMD:R_0805_2012Metric, symbol Device:R_Small
- added R12: 2M, Resistor_SMD:R_0805_2012Metric, symbol Device:R_Small
- added U2: MIC5365-3.3YD5, Package_TO_SOT_SMD:SOT-23-5, symbol Regulator_Linear:MIC5365-3.3YD5
- added U4: CP2104, Package_DFN_QFN:QFN-24-1EP_4x4mm_P0.5mm_EP2.6x2.6mm, symbol Interface_USB:CP2104
- added Y1: SIT1533AI-H4-DCC-32.768E, SamacSys_Parts:SIT1533AIH4DCC32768E, symbol SamacSys_Parts:SIT1533AI-H4-DCC-32.768E
- J11: value Conn_01x02_Male -> Conn_01x02
- R1, R2, R4: value 100 ohm -> 1k ohm
Connections:
- net +5V: now also U4.7 (REGIN), U4.8 (VBUS)
- net +BATT: now also R11.2
- net B2: now also U1.P7 (P0.26); no longer U1.P37 (P0.19)
- net B3: now also U1.P11 (P0.30/AIN6); no longer U1.P12 (P0.31/AIN7)
- net B5: now also U1.P9 (P0.28/AIN4); no longer U1.P11 (P0.30/AIN6)
- net B6: now also U1.P27 (P0.11); no longer U1.P26 (P0.10/NFC2)
- net C0: now also U1.P25 (P0.09/NFC1); no longer U1.P23 (P0.07)
- net D5: now also U1.P8 (P0.27); no longer U1.P35 (P0.17)
- net D6: now also U1.P26 (P0.10/NFC2); no longer U1.P24 (P0.08)
- net D7: now also U1.P23 (P0.07); no longer U1.P22 (P0.06)
- net GND: now also R1.1, R2.1, U1.P14 (P0.01/XL2), C5.2, C6.2, C8.2, R12.1, U2.2 (GND), U4.2 (GND), Y1.2 (GND)
- net RESET: now also C7.1
- net VCC: now also C6.1, U2.5 (VOUT), U4.5 (VIO), U4.6 (VDD), Y1.4 (VDD); no longer R1.1, R2.1
- net at U1.P13 (P0.00/XL1): now also Y1.3 (CLK_OUT)
- net D+: now reaches J12.A6 (DP1)
- net D+: now also J12.B6 (DP2), U4.3 (D+)
- net D-: now reaches J12.A7 (DN1)
- net D-: now also J12.B7 (DN2), U4.4 (D-)
- net at R1.2: now also D1.1 (K); no longer D1.2 (A)
- net at R2.2: now also D2.1 (K); no longer D2.2 (A)
- net at C1.1, D5.1 (K), Q1.2 (S): now also J14.1 (Pin_1), U2.1 (VIN)
- net P6: no longer names the net of U1.P6 (P0.25)
- removed net P7: D2.1 (K), U1.P7 (P0.26)
- removed net P8: D1.1 (K), U1.P8 (P0.27)
- new net: C5.1, U4.16 (VPP)
- new net: R10.1, U4.21 (TXD)
- new net: J14.2 (Pin_2), U2.3 (EN)
- new net BMonitor: C8.1, R11.1, R12.2, U1.P12 (P0.31/AIN7)
- new net DTR: C7.2, U4.23 (DTR)
- new net LED1: D2.2 (A), U1.P35 (P0.17)
- new net LED2: D1.2 (A), U1.P37 (P0.19)
- new net RXD: R10.2, U1.P24 (P0.08)
- new net TXD: U1.P22 (P0.06), U4.20 (RXD)
- no-connect marks 57 -> 52
Other:
- moved on the sheet: D1, D2

Commit message: pre-final
Parts:
- renumbered D4 to D3, D3 to D4, R4 to R3, R3 to R4
Connections:
- net +5V: no longer R3.1
- net GND: now also R3.1; no longer D3.1 (K)
- net LED1: now also D1.2 (A), U1.P37 (P0.19); no longer D2.2 (A), U1.P35 (P0.17)
- net LED2: now also D2.2 (A), U1.P35 (P0.17); no longer D1.2 (A), U1.P37 (P0.19)
- net VCC: no longer C6.1, U4.5 (VIO), U4.6 (VDD)
- net LED3: now reaches U1.P6 (P0.25)
- net LED3: now also D3.2 (A)
- net at R3.2: now also D3.1 (K); no longer D3.2 (A)
- new net: C6.1, U4.5 (VIO), U4.6 (VDD)
- no-connect marks 52 -> 66
Other:
- note added: "Key Matrix Connectors"
- note added: "LIPO Charging"
- note added: "LIPO Monitoring"
- note added: "Lights"
- note added: "Mounting Hole"
- note added: "Reset Circuit"
- note added: "SWD Headers"
- note added: "USB C"
- note added: "USB/UART"
- note added: "Voltage Regulation"
- note added: "nRF52832 Module"
- moved on the sheet: BT1, C3, C4, C5, C6, C7, C8, D1, D2, D3, D4, J1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

Commit message: readme update
Parts:
- removed J14: Conn_01x02, Connector_PinHeader_2.54mm:PinHeader_1x02_P2.54mm_Vertical, symbol Connector:Conn_01x02_Male
- removed U2: MIC5365-3.3YD5, Package_TO_SOT_SMD:SOT-23-5, symbol Regulator_Linear:MIC5365-3.3YD5
- added U2: MIC5504-3.3YM5, Package_TO_SOT_SMD:SOT-23-5, symbol Regulator_Linear:MIC5504-3.3YM5
Connections:
- net GND: now also U2.2 (GND)
- net VCC: now also U2.5 (VOUT)
- net at C1.1, D5.1 (K), Q1.2 (S): now also U2.1 (VIN), U2.3 (EN)
Changed lines of the file:
@@
-	1    0    0    -1
-$EndComp
-$Comp
-L Connector:Conn_01x02_Male J14
-U 1 1 5F2E5B27
-P 5200 1600
-F 0 "J14" H 5100 1600 50  0000 C CNN
-F 1 "Conn_01x02" H 5300 1400 50  0000 C CNN
-F 2 "Connector_PinHeader_2.54mm:PinHeader_1x02_P2.54mm_Vertical" H 5200 1600 50  0001 C CNN
-F 3 "~" H 5200 1600 50  0001 C CNN
-	1    5200 1600
 	1    0    0    -1
 $EndComp
@@
 	4950 1500 4950 1900
 Wire Wire Line
-	5400 1300 5400 1600
+	5400 1300 5400 1500
 Wire Wire Line
 	5400 1300 4950 1300
-Wire Wire Line
-	5500 1700 5400 1700
 Wire Wire Line
 	4950 1900 5900 1900
@@
 	5250 7950 5250 8100
 Wire Wire Line
-	5500 1500 5500 1700
-Wire Wire Line
 	5400 1300 5500 1300
 Connection ~ 5400 1300
@@
 	6300 1300 6500 1300
 Connection ~ 6500 1300
-$Comp
-L Regulator_Linear:MIC5365-3.3YD5 U2
-U 1 1 5F32FB87
-P 5900 1400
-F 0 "U2" H 5900 1767 50  0000 C CNN
-F 1 "MIC5365-3.3YD5" H 5900 1676 50  0000 C CNN
-F 2 "Package_TO_SOT_SMD:SOT-23-5" H 5900 1750 50  0001 C CNN
-F 3 "http://ww1.microchip.com/downloads/en/DeviceDoc/mic5365.pdf" H 5650 1650 50  0001 C CNN
-	1    5900 1400
-	1    0    0    -1
-$EndComp
-Connection ~ 5900 1700
 Wire Notes Line
 	450  6400 3700 6400
@@
 Wire Wire Line
 	2200 2000 2200 2100
-NoConn ~ 1650 9800
 NoConn ~ 13600 3750
 NoConn ~ 12800 8050
@@
 Text Notes 8250 3350 0    50   ~ 0
 nRF52832 Module
+$Comp
+L Regulator_Linear:MIC5504-3.3YM5 U2
+U 1 1 5F408DEA
+P 5900 1400
+F 0 "U2" H 5900 1767 50  0000 C CNN
+F 1 "MIC5504-3.3YM5" H 5900 1676 50  0000 C CNN
+F 2 "Package_TO_SOT_SMD:SOT-23-5" H 5900 1000 50  0001 C CNN
+F 3 "http://ww1.microchip.com/downloads/en/DeviceDoc/MIC550X.pdf" H 5650 1650 50  0001 C CNN
+	1    5900 1400
+	1    0    0    -1
+$EndComp
+Connection ~ 5900 1700
+Wire Wire Line
+	5500 1500 5400 1500
+NoConn ~ 1650 9800
 $EndSCHEMATC

Commit message: Final Gerbers and BOM
Parts:
- added J14: Conn_01x02, Connector_PinHeader_2.54mm:PinHeader_1x02_P2.54mm_Vertical, symbol Connector:Conn_01x02_Male
Connections:
- net at C1.1, D5.1 (K), Q1.2 (S)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: now also J14.1 (Pin_1); no longer U2.3 (EN)
- new net: J14.2 (Pin_2), U2.3 (EN)
Changed lines of the file:
@@
 	4950 1500 4950 1900
-Wire Wire Line
-	5400 1300 5400 1500
-Wire Wire Line
-	5400 1300 4950 1300
 Wire Wire Line
 	4950 1900 5900 1900
@@
 Wire Wire Line
 	5250 7950 5250 8100
-Wire Wire Line
-	5400 1300 5500 1300
-Connection ~ 5400 1300
 Wire Wire Line
 	6300 1300 6500 1300
@@
 $EndComp
 Connection ~ 5900 1700
+NoConn ~ 1650 9800
+Wire Wire Line
+	4950 1300 5300 1300
+$Comp
+L Connector:Conn_01x02_Male J14
+U 1 1 5F549B61
+P 5300 1800
+F 0 "J14" V 5454 1612 50  0000 R CNN
+F 1 "Conn_01x02" V 5250 1700 50  0000 R CNN
+F 2 "Connector_PinHeader_2.54mm:PinHeader_1x02_P2.54mm_Vertical" H 5300 1800 50  0001 C CNN
+F 3 "~" H 5300 1800 50  0001 C CNN
+	1    5300 1800
+	0    -1   -1   0
+$EndComp
 Wire Wire Line
 	5500 1500 5400 1500
-NoConn ~ 1650 9800
+Wire Wire Line
+	5400 1500 5400 1600
+Wire Wire Line
+	5300 1600 5300 1300
+Connection ~ 5300 1300
+Wire Wire Line
+	5300 1300 5500 1300
 $EndSCHEMATC

Commit message: Rev 0a board complete
Connections:
- net C6: now also J7.7 (Pin_7)
- no-connect marks 66 -> 65
Changed lines of the file:
@@
 NoConn ~ 14900 4450
 NoConn ~ 15400 4550
-NoConn ~ 15400 4250
 NoConn ~ 15400 4350
 NoConn ~ 15400 5450
@@
 Wire Wire Line
 	5300 1300 5500 1300
+Text GLabel 15400 4250 2    50   Input ~ 0
+C6
 $EndSCHEMATC
